File: Ignition.kicad_sch (KiCad schematic)
At the start: 2 parts, among them Q1 Q_NIGBT_GCE

Commit message: a lot of changes
Parts:
- Q5: renamed from Q1; value Q_NIGBT_GCE -> RGPR30BM40HRTL
- R9: renamed from R1; footprint Resistor_SMD:R_0603_1608Metric -> Resistor_SMD:R_0402_1005Metric; MPN AC0603JR-071KL -> AC0402FR-071KL
