File: Injection.kicad_sch (KiCad schematic)
At the start: 3 parts, among them Q3 Q_NMOS_GDS

Commit message: a lot of changes
Parts:
- Q1: renamed from Q3; value Q_NMOS_GDS -> VND14NV04TR-E
- R1: renamed from R3; footprint Resistor_SMD:R_0603_1608Metric -> Resistor_SMD:R_0402_1005Metric; MPN (none) -> AC0402FR-07330RL
- R2: renamed from R4; footprint Resistor_SMD:R_0603_1608Metric -> Resistor_SMD:R_0402_1005Metric; MPN (none) -> AC0402FR-0768KL
