File: Outputs.kicad_sch (KiCad schematic)
At the start: 0 parts

Commit message: a lot of changes
Parts:
- added C1, C10, C2, C3, C9: 10nF, Capacitor_SMD:C_0402_1005Metric, symbol Device:C
- added C4, C5, C8: 100nF, Capacitor_SMD:C_0402_1005Metric, symbol Device:C
- added C6: 100uF, Capacitor_SMD:CP_Elec_8x10, symbol Device:C_Polarized_Small
- added C7: 1uF, Capacitor_SMD:C_0805_2012Metric, symbol Device:C
- added D1, D2, D3, D4: NSVRB751V40T1G, Diode_SMD:D_SOD-323, symbol Diode:1N4148WS
- added D5, D6: MMSZ4688-TP, Diode_SMD:D_SOD-123, symbol Device:D_Zener
- added F1, F2, F3, F4, F5: 350 mA, Fuse:Fuse_1206_3216Metric, symbol Device:Polyfuse
- added Q10, Q11, Q7, Q8, Q9: PJA3460, Package_TO_SOT_SMD:SOT-23-3, symbol Device:Q_NMOS_GDS
- added R11: 10k, Resistor_SMD:R_1206_3216Metric, symbol Device:R
- added R12, R13, R14, R15, R23: 330, Resistor_SMD:R_0402_1005Metric, symbol Device:R
- added R16, R17, R18, R19, R25: 68k, Resistor_SMD:R_0402_1005Metric, symbol Device:R
- added R20, R21, R22: 33k, Resistor_SMD:R_0402_1005Metric, symbol Device:R
- added R24: 100k, Resistor_SMD:R_0402_1005Metric, symbol Device:R
- added R26: 4k7, Resistor_SMD:R_0402_1005Metric, symbol Device:R
- added U1: TLE9201SG, footprints:Infineon_PG-DSO-12-17_ThermalVias, symbol tle9201:TLE9201SG
Connections:
- new net: Q8.1 (G), R13.2, R17.2
- new net: F2.1, Q8.2 (D), R11.1
- new net: F3.1, Q9.2 (D)
- new net: D2.1 (K), D4.1 (K), D6.1 (K), R23.1
- new net: C1.2, D2.2 (A), R20.1
- new net: C3.1, D3.2 (A), R22.1
- new net: F1.1, Q7.2 (D), R20.2, R21.2
- new net: Q11.1 (G), R23.2, R25.2
- new net: C2.1, D1.2 (A), R21.1
- new net: Q7.1 (G), R12.2, R16.2
- new net: Q9.1 (G), R14.2, R18.2
- new net: F4.1, Q10.2 (D)
- new net: Q10.1 (G), R15.2, R19.2
- new net 12V_Fused: C6.1, C7.1, C8.1, R11.2, U1.4 (VS)
- new net 12V_PERM: F5.1, Q11.2 (D)
- new net 3V3: C5.1, R26.1, U1.2 (VSO)
- new net DIR: U1.1 (DIR)
- new net DIS: R26.2, U1.11 (DIS)
- new net ETB1: C9.1, U1.5 (OUT1)
- new net ETB2: C10.1, U1.7 (OUT2)
- new net FAN: R15.1
- new net FAN_OUT: F4.2
- new net FPUMP: R12.1, R22.2
- new net FPUMP_OUT: F1.2
- new net GND: C1.1, C10.2, C2.2, C3.2, C4.2, C5.2, C6.2, C7.2, C8.2, C9.2, D5.2 (A), D6.2 (A), Q10.3 (S), Q11.3 (S), Q7.3 (S), Q8.3 (S), Q9.3 (S), R16.1, R17.1, R18.1, R19.1, R24.1, R25.1, U1.10 (SCK), U1.13 (GND), U1.6 (GND), U1.8 (SI), U1.9 (CSN)
- new net IGN_OUT: C4.1, D1.1 (K), D3.1 (K), D5.1 (K), R24.2
- new net MAIN_RELAY_OUT: F5.2
- new net MAIN_RELAY_UC: D4.2 (A)
- new net MIL: R14.1
- new net MIL_OUT: F3.2
- new net PWM: U1.12 (PWM)
- new net TACHO: R13.1
- new net TACHO_OUT: F2.2
- no-connect marks 0 -> 1
