File: balefi.kicad_sch (KiCad schematic)
At the start: 2 parts, among them J1 Connectors_EFI_ECUs_Con_82521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, M2 Module:mega-mcu100/0.3

Commit message: Started designing schematic
Parts:
- added H1, H2: MountingHole_Pad, MountingHole:MountingHole_3.7mm_Pad_Via, symbol Mechanical:MountingHole_Pad
- added H3: MountingHole, MountingHole:MountingHole_3.7mm, symbol Mechanical:MountingHole
- added M1: Module-knock-0.2, hellen-one-knock-0.2:knock, symbol hellen-one-knock-0.2:Module-knock-0.2
- added M3, M4: Module-vr-discrete-0.4, hellen-one-vr-discrete-0.4:vr-discrete, symbol hellen-one-vr-discrete-0.4:Module-vr-discrete-0.4
- J1: footprint rusefi_lib:825213-1 -> rusefi_lib:825213-1_FIAT
Connections:
- net +5VA: now reaches M2.E1 (V5A_SWITCHABLE)
- net +5VA: now also M2.W14 (V5A_SWITCHABLE), M2.W2 (V5A_SWITCHABLE), M1.E1 (V5A), M3.E4 (V5_IN), M4.E4 (V5_IN)
- net MIL_UC: now reaches M2.E10 (OUT_INJ8_(PD12))
- net TACHO_UC: now reaches M2.E11 (OUT_INJ7_(PD15))
- net FAN_UC: now reaches M2.E12 (OUT_INJ6_(PA8))
- net BOOST_UC: now reaches M2.E13 (OUT_INJ5_(PD2))
- net INJ4_UC: now reaches M2.E14 (OUT_INJ4_(PD10))
- net INJ3_UC: now reaches M2.E15 (OUT_INJ3_(PD11))
- net INJ2_UC: now reaches M2.E16 (OUT_INJ2_(PA9))
- net INJ1_UC: now reaches M2.E17 (OUT_INJ1_(PD3))
- net FPUMP_UC: now reaches M2.E18 (OUT_PWM1_(PD13))
- net GNDA: now reaches M2.E2 (GNDA)
- net GNDA: now also M2.W1 (GNDA)
- net VR_THRESHOLD: now reaches M2.E23 (OUT_PWM6_(PD14))
- net VR_THRESHOLD: now also M3.E1 (Thresh_IN), M4.E1 (Thresh_IN)
- net VIGN: now reaches M2.E5 (IN_VIGN_(PA5))
- net GND: now reaches M2.G (GND)
- net GND: now also M1.E2 (GND), M3.G (GND), M4.G (GND)
- net VBUS: now reaches M2.N1 (VBUS)
- net BT_RX: now reaches M2.N13 (UART2_TX_(PD5))
- net BT_TX: now reaches M2.N14 (UART2_RX_(PD6))
- net +3.3VA: now reaches M2.N15 (V33_SWITCHABLE)
- net VBAT: now reaches M2.N17 (VBAT)
- net USBM: now reaches M2.N2 (USBM_(PA11))
- net PWR_EN: now reaches M2.N20 (OUT_PWR_EN_(PE10))
- net +3.3V: now reaches M2.N21 (V33)
- net +3.3V: now also M2.N23 (V33)
- net USBP: now reaches M2.N3 (USBP_(PA12))
- net SWDIO: now reaches M2.N5 (SWDIO_(PA13))
- net SWCLK: now reaches M2.N6 (SWCLK_(PA14))
- net ~{RESET}: now reaches M2.N7 (nReset)
- net FUEL_PRESS: now reaches M2.S12 (IN_MAP2_(PC1))
- net FUEL_PRESS: now also J1.24
- net MAP: now reaches M2.S13 (IN_MAP1_(PC0))
- net MAP: now also J1.32
- net CRANK_UC: now reaches M2.S14 (IN_CRANK_(PB1))
- net CRANK_UC: now also M4.E3 (OUT)
- net KNOCK_UC: now reaches M2.S15 (IN_KNOCK_(PA2))
- net KNOCK_UC: now also M1.E3 (OUT_KNOCK)
- net CAM_UC: now reaches M2.S16 (IN_CAM_(PA6))
- net CAM_UC: now also M3.E3 (OUT)
- net VSS_UC: now reaches M2.S17 (IN_VSS_(PE11))
- net TPS: now reaches M2.S18 (IN_TPS_(PA4))
- net TPS: now also J1.30
- net PPS1_IN: now reaches M2.S19 (IN_PPS_(PA3))
- net PPS1_IN: now also J1.27
- net IAT: now reaches M2.S20 (IN_IAT_(PC3))
- net IAT: now also J1.31
- net CLT: now reaches M2.S21 (IN_CLT_(PC2))
- net CLT: now also J1.13
- net VREF1: now reaches M2.S22 (VREF1)
- net VREF1: now also M1.W2 (VREF)
- net VMAIN_UC: now reaches M2.S6 (IN_AUX4_(PC5))
- net OIL_TEMP: now reaches M2.S7 (IN_AUX3_(PA7))
- net OIL_TEMP: now also J1.25
- net PPS2_IN: now reaches M2.S8 (IN_AUX2_(PC4/PE9))
- net PPS2_IN: now also J1.9
- net OIL_PRESS: now reaches M2.S9 (IN_AUX1_(PB0))
- net OIL_PRESS: now also J1.8
- net IGN1_UC: now reaches M2.W10 (IGN1_(PC13))
- net CANH: now reaches M2.W11 (CANH)
- net CANH: now also J1.15
- net CANL: now reaches M2.W12 (CANL)
- net CANL: now also J1.10
- net IGN2_UC: now reaches M2.W9 (IGN2_(PE5))
- net IGN14: now reaches J1.1
- net CRANK-: now reaches J1.11
- net CRANK-: now also M4.W1 (VR-)
- net AGND: now reaches J1.12
- net AGND: now also J1.16
- net 5VP: now reaches J1.14
- net PGND: now reaches J1.17
- net INJ1: now reaches J1.18
- net IGN23: now reaches J1.19
- net ETB2: now reaches J1.2
- net ETB1: now reaches J1.20
- net INJ3: now reaches J1.21
- net TACHO_OUT: now reaches J1.22
- net FPUMP_RELAY: now reaches J1.23
- net IGNITION: now reaches J1.26
- net CRANK+: now reaches J1.28
- net CRANK+: now also M4.W2 (VR+)
- net KNOCK_IN: now reaches J1.29
- net KNOCK_IN: now also M1.W1 (IN_KNOCK)
- net FAN_OUT: now reaches J1.3
- net CAM-: now reaches J1.33
- net CAM-: now also M3.W1 (VR-)
- net CAM+: now reaches J1.34
- net CAM+: now also M3.W2 (VR+)
- net INJ2: now reaches J1.35
- net INJ4: now reaches J1.4
- net BOOST_OUT: now reaches J1.5
- net MIL: now reaches J1.6
- net VSS: now reaches J1.7
- no-connect marks 14 -> 28
Other:
- added sheet Ignition1 (Ignition.kicad_sch)
- added sheet Ignition2 (Ignition.kicad_sch)
- added sheet Injection1 (Injection.kicad_sch)
- added sheet Injection2 (Injection.kicad_sch)
- added sheet Injection3 (Injection.kicad_sch)
- added sheet Injection4 (Injection.kicad_sch)
- added sheet Outputs (Outputs.kicad_sch)
- note added: "Input"
- note added: "Power"
- note added: "VND5N07TR-E"
- moved on the sheet: J1, M2

Commit message: a lot of changes
Parts:
- removed M1: Module-knock-0.2, hellen-one-knock-0.2:knock, symbol hellen-one-knock-0.2:Module-knock-0.2
- removed M2: Module:mega-mcu100/0.3, hellen-one-mega-mcu100-0.3:mega-mcu100, symbol mega-mcu100_0.3:Module{colon}mega-mcu100/0.3
- removed M3, M4: Module-vr-discrete-0.4, hellen-one-vr-discrete-0.4:vr-discrete, symbol hellen-one-vr-discrete-0.4:Module-vr-discrete-0.4
- added NT1: NetTie_2, NetTie:NetTie-2_SMD_Pad2.0mm, symbol Device:NetTie_2
- H1: renamed from H3; now not fitted
- H2: now not fitted
- H3: renamed from H1; now not fitted
- J1: symbol auto_connectors:Connectors_EFI_ECUs_Con_825213-1 -> balefi-library:Connectors_EFI_ECUs_Con_825213-1
Connections:
- net AGND is gone; now on net GNDA: J1.12, J1.16
- net FUEL_PRESS is gone; now on net INJ2: J1.24
- net OIL_PRESS is gone; now on net INJ4: J1.8
- net PGND is gone; now on net GND: J1.17
- net GND: now also H2.1, H3.1, NT1.1
- net GNDA: now also NT1.2
- net INJ2: no longer J1.35
- net INJ4: no longer J1.4
- net BOOST_OUT renamed TPS2
- net CAM- renamed CAM-/HALL
- net IGNITION renamed EGT+
- net OIL_TEMP renamed EGT-
- net TPS renamed TPS1
- new net 12V_RAW: J1.35
- new net MAIN_RELAY: J1.4
- no-connect marks 28 -> 2
Other:
- added sheet Frequency_inputs (Freq_inputs.kicad_sch)
- added sheet Knock (Knock.kicad_sch)
- added sheet MCU_module (MCU_module.kicad_sch)
- added sheet Power (Power.kicad_sch)
- sheet Outputs ports: added 12V_Fused, 12V_PERM, 3V3, DIR, DIS, ETB1, ETB2, FAN, FAN_OUT, FPUMP, FPUMP_OUT, IGN_OUT, MAIN_RELAY_OUT, MAIN_RELAY_UC, MIL, MIL_OUT, PWM, TACHO, TACHO_OUT; removed none
- note removed: "Input"
- note removed: "VND5N07TR-E"
